File: HunterCat-NFC/HunterCat-NFC.sch (KiCad schematic (older format))
At the start: 64 parts, among them J1 Battery, P1 USB_C_Plug_USB2.0, SW1 RESET, U1 ATSAMD21E18A, U2 PN7150B0HN/C11004, U3 MCP73831-3-OT, U4 AP2112K-3.3, U5 W25Q32JVSS, Y1 27.12Mhz

Commit message: alpha version
Parts:
- C1, C10, C11, C12, C13, C14, C15, C16, C17, C18, C19, C2, C20, C21, C22, C23, C24, C3, C4, C5, C6, C7, C8, C9: footprint (none) -> Capacitor_SMD:C_0805_2012Metric_Pad1.15x1.40mm_HandSolder
- D1, D2, D3, D4: footprint (none) -> LED_SMD:LED_0805_2012Metric_Pad1.15x1.40mm_HandSolder
- JP1, JP2: footprint (none) -> Jumper:SolderJumper-3_P1.3mm_Bridged12_RoundedPad1.0x1.5mm
- L1, L2, L3: footprint (none) -> Inductor_SMD:L_0805_2012Metric_Pad1.15x1.40mm_HandSolder
- R1, R10, R11, R12, R13, R16, R17, R18, R19, R2, R20, R21, R3, R4, R5, R6, R7, R8, R9: footprint (none) -> Resistor_SMD:R_0805_2012Metric_Pad1.15x1.40mm_HandSolder
- R14, R15: value R_Small -> 0; footprint (none) -> Resistor_SMD:R_0805_2012Metric_Pad1.15x1.40mm_HandSolder
- U2: footprint QFN50P600X600X100-41N -> Package_DFN_QFN:QFN-40-1EP_6x6mm_P0.5mm_EP4.6x4.6mm; symbol PN7150B0HN_C11002E:PN7150B0HN_C11002E -> HunterCat-NFC-rescue:PN7150B0HN_C11002E-PN7150B0HN_C11002E

Commit message: Update libraries, add antenna 30x30mm
Parts:
- removed U2: PN7150B0HN/C11004, Package_DFN_QFN:QFN-40-1EP_6x6mm_P0.5mm_EP4.6x4.6mm, symbol HunterCat-NFC-rescue:PN7150B0HN_C11002E-PN7150B0HN_C11002E
- added U2: PN7150B0HN_C11002E-PN7150B0HN_C11002E, Package_DFN_QFN:QFN-40-1EP_6x6mm_P0.5mm_EP4.6x4.6mm, symbol hunter-cat-nfc:PN7150B0HN_C11002E-PN7150B0HN_C11002E
- C10, C11, C12, C13, C14, C15, C17, C18, C19, C20, C21, C22: footprint Capacitor_SMD:C_0805_2012Metric_Pad1.15x1.40mm_HandSolder -> Capacitor_SMD:C_0603_1608Metric_Pad1.05x0.95mm_HandSolder
- L1, L2: footprint Inductor_SMD:L_0805_2012Metric_Pad1.15x1.40mm_HandSolder -> Inductor_SMD:L_0603_1608Metric_Pad1.05x0.95mm_HandSolder
- L3: footprint Inductor_SMD:L_0805_2012Metric_Pad1.15x1.40mm_HandSolder -> hunter-cat-nfc:NFC-antenna30.4x30.4mm
- P1: footprint (none) -> Connectors:C393939
- R11, R13: footprint Resistor_SMD:R_0805_2012Metric_Pad1.15x1.40mm_HandSolder -> Resistor_SMD:R_0603_1608Metric_Pad1.05x0.95mm_HandSolder
- R14, R15: value 0 -> 3.24R; footprint Resistor_SMD:R_0805_2012Metric_Pad1.15x1.40mm_HandSolder -> Resistor_SMD:R_0603_1608Metric_Pad1.05x0.95mm_HandSolder
- SW1: footprint (none) -> Button_Switch_SMD:SW_SPST_TL3342
- U1: symbol Electronic_Cats:ATSAMD21E18A -> HunterCat-NFC-rescue:ATSAMD21E18A-Electronic_Cats
Connections:
- net +3V3: now also U2.13 (VBAT1), U2.6 (VDD(PAD))
- net +BATT: now also U2.12 (VBAT2), U2.26 (VBAT)
- net ADR0: now also U2.1 (I2CADR0)
- net ADR1: now also U2.3 (I2CADR1)
- net CLK: now also U2.40 (CLK_REQ)
- net GND: now also U2.19 (VSS(TX)), U2.2 (VSS), U2.27 (VSS), U2.4 (VSS(PAD)), U2.41 (VSS), U2.9 (VSS)
- net IRQ: now also U2.8 (IRQ)
- net RXN: now also U2.15 (RXN)
- net RXP: now also U2.16 (RXP)
- net SCL: now also U2.7 (I2CSCL)
- net SDA: now also U2.5 (I2CSDA)
- net TX1: now also U2.21 (TX1)
- net TX2: now also U2.18 (TX2)
- net VEN: now also U2.10 (VEN)
- net at C8.1: now also U2.14 (VDD(TX)), U2.22 (VDD(TX_IN))
- net at C7.1: now also U2.17 (VDD(MID))
- net at C5.1: now also U2.28 (VDDA), U2.29 (VDD), U2.30 (VDDD)
- net at C4.1, Y1.1: now also U2.36 (NFC_CLK_XTAL1); no longer C3.1
- net at Y1.3: now also C3.1, U2.37 (NFC_CLK_XTAL2)
- net at C14.1, C15.1, C19.1: now also C21.1, R14.2
- no-connect marks 11 -> 10
Other:
- note added: "ANTENA\n30.4mm\n"
- note removed: "ANTENA"
