File: HunterCat-NFC/HunterCat-NFC.kicad_pcb (KiCad board)
At the start: 2 copper layers, 108 x 53.8 mm, 66 parts, among them J1 Battery, J2 Breakout Conn, P1 USB_C_Plug_USB2.0, SW1 RESET, U1 ATSAMD21E18A, U2 PN7150B0HN_C11002E-PN7150B0HN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, U3 MCP73831-3-OT, U4 AP2112K-3.3, U5 W25Q32JVSS, Y1 27.12Mhz

Commit message: value c25
Parts:
- C25: value 10uF -> 0.1uF
Changed lines of the file:
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@@
       (effects (font (size 1 1) (thickness 0.15)))
     )
-    (fp_text value 10uF (at 0 1.65) (layer F.Fab)
+    (fp_text value 0.1uF (at 0 1.65) (layer F.Fab)
       (effects (font (size 1 1) (thickness 0.15)))
     )
