File: HunterCat-NFC/HunterCat-NFC/HunterCat-NFC.sch (KiCad schematic (older format))
At the start: 64 parts, among them J1 Battery, J2 Conn_01x06_Female, P1 USB_C_Plug_USB2.0, Q1 DMG3415U-7, SW1 RESET, SW2 GPIO, SW3 GPIO1, SW4 GPIO2, U1 ATSAMD21E18A, U2 PN7150B0HN_C11002E-PN7150B0HN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

Commit message: fix mosfet and battery voltage
Parts:
- removed Q1: DMG3415U-7, Package_TO_SOT_SMD:TSOT-23, symbol Transistor_FET:BS107
- added Q?: DMG3415U-7, Package_TO_SOT_THT:TO-92L_Inline, symbol Transistor_FET:TP0610L
Connections:
- net +3V3: now also C9.1, U2.12 (VBAT2), U2.26 (VBAT)
- net +BATT: now also Q?.3 (D); no longer C9.1, U2.12 (VBAT2), U2.26 (VBAT)
- net VBUS: now also Q?.2 (G)
- net at C23.1, D5.1 (K), R16.1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: now also Q?.1 (S)
Changed lines of the file:
@@
 Sheet 1 1
 Title "Hunter Cat NFC"
-Date "2020-07-28"
-Rev "1.1"
+Date "2020-10-05"
+Rev "1.2"
 Comp "Electronic Cats"
 Comment1 ""
@@
 	9375 4335 9375 4285
 $Comp
-L Transistor_FET:BS107 Q1
-U 1 1 5F2FE16A
-P 9275 4085
-F 0 "Q1" H 9479 4131 50  0000 L CNN
-F 1 "DMG3415U-7" H 9479 4040 50  0000 L CNN
-F 2 "Package_TO_SOT_SMD:TSOT-23" H 9475 4010 50  0001 L CIN
-F 3 "http://www.onsemi.com/pub_link/Collateral/BS107-D.PDF" H 9275 4085 50  0001 L CNN
-	1    9275 4085
-	1    0    0    -1
-$EndComp
-$Comp
 L Diode:MBR340 D5
 U 1 1 5F318682
@@
 L power:+3V3 #PWR017
 U 1 1 5E819D40
-P 5225 1440
-F 0 "#PWR017" H 5225 1290 50  0001 C CNN
-F 1 "+3V3" H 5240 1613 50  0000 C CNN
-F 2 "" H 5225 1440 50  0001 C CNN
-F 3 "" H 5225 1440 50  0001 C CNN
-	1    5225 1440
-	1    0    0    -1
-$EndComp
-Wire Wire Line
-	4890 1340 5055 1340
-Connection ~ 4890 1340
-Wire Wire Line
-	4890 1540 4920 1540
-Connection ~ 4890 1540
-Wire Wire Line
-	3460 1540 4890 1540
-Wire Wire Line
-	4890 1540 4890 1340
-$Comp
-L power:+BATT #PWR016
-U 1 1 5E8068AB
 P 5055 1340
-F 0 "#PWR016" H 5055 1190 50  0001 C CNN
-F 1 "+BATT" H 5070 1513 50  0000 C CNN
+F 0 "#PWR017" H 5055 1190 50  0001 C CNN
+F 1 "+3V3" H 5070 1513 50  0000 C CNN
 F 2 "" H 5055 1340 50  0001 C CNN
 F 3 "" H 5055 1340 50  0001 C CNN
@@
 $EndComp
 Wire Wire Line
-	3460 1440 5225 1440
+	4890 1340 5055 1340
+Connection ~ 4890 1340
+Wire Wire Line
+	4890 1540 4920 1540
+Connection ~ 4890 1540
+Wire Wire Line
+	3460 1540 4890 1540
 Wire Wire Line
 	3460 1340 4890 1340
@@
 	3255 7210 3150 7210
 NoConn ~ 3150 4710
+Wire Wire Line
+	4890 1540 4890 1440
+Wire Wire Line
+	3460 1440 4890 1440
+Connection ~ 4890 1440
+Wire Wire Line
+	4890 1440 4890 1340
+$Comp
+L Transistor_FET:TP0610L Q?
+U 1 1 5F7FE226
+P 9275 4085
+F 0 "Q?" H 9479 4131 50  0000 L CNN
+F 1 "DMG3415U-7" H 9479 4040 50  0000 L CNN
+F 2 "Package_TO_SOT_THT:TO-92L_Inline" H 9475 4010 50  0001 L CIN
+F 3 "http://www.vishay.com/docs/70209/70209.pdf" H 9275 4085 50  0001 L CNN
+	1    9275 4085
+	1    0    0    -1
+$EndComp
 $EndSCHEMATC

Commit message: update v1.1 2 layes
Parts:
- removed Q?: DMG3415U-7, Package_TO_SOT_THT:TO-92L_Inline, symbol Transistor_FET:TP0610L
- added Q1: DMG3415U-7, Package_TO_SOT_SMD:SOT-23, symbol Device:Q_PMOS_GSD
Connections:
- net +BATT: now also Q1.3 (D)
- net VBUS: now also Q1.1 (G)
- net at C23.1, D5.1 (K), R16.1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: now also Q1.2 (S)
Changed lines of the file:
@@
 U 1 1 5F318682
 P 9170 4335
-F 0 "D5" H 9170 4118 50  0000 C CNN
-F 1 "MBR120" H 9170 4209 50  0000 C CNN
+F 0 "D5" H 9295 4295 50  0000 C CNN
+F 1 "MBR120" H 9205 4455 50  0000 C CNN
 F 2 "Diode_SMD:D_SOD-123F" H 9170 4160 50  0001 C CNN
 F 3 "http://www.onsemi.com/pub_link/Collateral/MBR340-D.PDF" H 9170 4335 50  0001 C CNN
@@
 	4890 1440 4890 1340
 $Comp
-L Transistor_FET:TP0610L Q?
-U 1 1 5F7FE226
+L Device:Q_PMOS_GSD Q1
+U 1 1 5FE5BD93
 P 9275 4085
-F 0 "Q?" H 9479 4131 50  0000 L CNN
-F 1 "DMG3415U-7" H 9479 4040 50  0000 L CNN
-F 2 "Package_TO_SOT_THT:TO-92L_Inline" H 9475 4010 50  0001 L CIN
-F 3 "http://www.vishay.com/docs/70209/70209.pdf" H 9275 4085 50  0001 L CNN
+F 0 "Q1" H 9435 4285 50  0000 L CNN
+F 1 "DMG3415U-7" H 9445 4200 50  0000 L CNN
+F 2 "Package_TO_SOT_SMD:SOT-23" H 9475 4185 50  0001 C CNN
+F 3 "https://www.mouser.mx/datasheet/2/115/ds31735-64958.pdf" H 9275 4085 50  0001 C CNN
 	1    9275 4085
 	1    0    0    -1

Commit message: add logos and mounitng holes again
Parts:
- added H1, H2, H3, H4: MountingHole, MountingHole:MountingHole_2.2mm_M2, symbol Mechanical:MountingHole
- added SW?: ON, symbol Switch:SW_SPST
Connections:
- net at C23.1, R16.1, U4.1 (VIN): now also SW?.2 (B); no longer D5.1 (K), Q1.2 (S)
- new net: D5.1 (K), Q1.2 (S), SW?.1 (A)
Other:
- moved on the sheet: C23, C24, D5, Q1, R16, R6, U4
