File: HunterCat-NFC/HunterCat-NFC/HunterCat-NFC.sch (KiCad schematic (older format))
At the start: 69 parts, among them J1 Battery, J2 Conn_01x06_Female, P1 USB_C_Plug_USB2.0, Q1 DMG3415U-7, SW1 RESET, SW2 GPIO, SW3 GPIO1, SW4 GPIO2, U1 ATSAMD21E18A, U2 PN7150B0HN_C11002E-PN7150B0HN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

Commit message: update traces
Parts:
- gave numbers to parts that had none: 1
Changed lines of the file:
@@
 $EndComp
 $Comp
-L Switch:SW_SPST SW?
+L Switch:SW_SPST SW5
 U 1 1 5F926B9C
 P 9480 4315
-F 0 "SW?" H 9480 4235 50  0000 C CNN
+F 0 "SW5" H 9480 4235 50  0000 C CNN
 F 1 "ON" H 9480 4459 50  0000 C CNN
 F 2 "hunter-cat-nfc:Micro_interruptor_SPDT" H 9480 4315 50  0001 C CNN

Commit message: update BOM
Parts:
- C1, C25, C7, C9: LCSC# (none) -> C387984; provedor (none) -> LCSC
- C10, C11, C12, C13, R14, R15: provedor (none) -> MOUSER
- C14: value 56pF/50V -> 100pF/50V; manf# GRM0335C1H560FA01D -> 06035A101JAT4A; provedor (none) -> MOUSER
- C16, C23, C24: LCSC# (none) -> C326057; provedor (none) -> LCSC
- C18: value 56pF -> 100pF/50V; manf# GRM0335C1H560FA01D -> 06035A101JAT4A; provedor (none) -> MOUSER
- C19, C20, C3, C4: provedor (none) -> LCSC
- C2, C5, C6, C8: LCSC# (none) -> C26413; provedor (none) -> LCSC
- D1: LCSC# (none) -> C130114; manf# R080508L3 -> -; provedor (none) -> LCSC
- D2: LCSC# (none) -> C205441; manf# ORH-B35A -> -; provedor (none) -> LCSC
- D3: LCSC# (none) -> C205442; manf# ORH-B35A -> -; provedor (none) -> LCSC
- D4: LCSC# (none) -> C84261; manf# 2012HYK-588J -> -; provedor (none) -> LCSC
- D5: LCSC# (none) -> C723989; manf# (none) -> -; provedor (none) -> LCSC
- F1, U1, U2, U3, U4, U5, Y1: LCSC# (none) -> -; provedor (none) -> MOUSER
- H1, H2, H3, H4, J1, J2, L3, SW5: LCSC# (none) -> -; manf# (none) -> -; provedor (none) -> -
- L1, L2: LCSC# (none) -> C434822; provedor (none) -> LCSC
- P1: LCSC# (none) -> C393939; manf# TYPE-C16PIN -> -; provedor (none) -> LCSC
- Q1: LCSC# (none) -> C96616; manf# (none) -> -; provedor (none) -> LCSC
- R1, R16, R2, R21: LCSC# (none) -> C15401; manf# CRCW080510K0JNEAC -> -; provedor (none) -> LCSC
- R10, R12, R17, R18, R4: LCSC# (none) -> C517454; provedor (none) -> LCSC
- R11, R13: LCSC# (none) -> C217937; provedor (none) -> LCSC
- R19, R20: value 100k -> 100K; LCSC# (none) -> C15458; provedor (none) -> LCSC
- R3, R5: LCSC# (none) -> C15458; manf# CRCW0805100KFKEAC -> ERJ6RBD1003V; provedor (none) -> LCSC
- R6: LCSC# (none) -> C15458; manf# (none) -> ERJ6RBD1003V; provedor (none) -> LCSC
- R8, R9: LCSC# (none) -> C131715; provedor (none) -> LCSC
- SW1, SW2, SW3, SW4: LCSC# (none) -> C318890; manf# TS-1187A-C-C-B -> -; provedor (none) -> LCSC

Commit message: update v1.2 footprint
Parts:
- U5: footprint USON:USON-8 -> hunter-cat-nfc:PSON50P200X300X50-9N
Changed lines of the file:
@@
 F 0 "U5" H 7091 6220 50  0000 C CNN
 F 1 "GD25Q16CEIGR" H 7719 6227 50  0000 C CNN
-F 2 "USON:USON-8" H 7360 5858 50  0001 C CNN
+F 2 "hunter-cat-nfc:PSON50P200X300X50-9N" H 7360 5858 50  0001 C CNN
 F 3 "https://www.mouser.com/ProductDetail/GigaDevice/GD25Q16CEIGR?qs=%2Fha2pyFadugslouyc%2Fmu%252BU7keVd3t830A8Tn7Tz5TRGEFPMfPa%252B4Kw%3D%3D" H 7360 5858 50  0001 C CNN
 F 4 "GD25Q16CEIGR" H 7360 5858 50  0001 C CNN "manf#"

Commit message: Sch
Parts:
- J1: footprint Connector_PinSocket_2.54mm:PinSocket_2x01_P2.54mm_Vertical -> Connector_PinSocket_2.54mm:PinSocket_2x01_P2.54mm_Vertical_SMD
Changed lines of the file:
@@
 F 0 "J1" H 8165 4257 50  0000 L CNN
 F 1 "Battery" H 8165 4166 50  0000 L CNN
-F 2 "Connector_PinSocket_2.54mm:PinSocket_2x01_P2.54mm_Vertical" H 8085 4265 50  0001 C CNN
+F 2 "Connector_PinSocket_2.54mm:PinSocket_2x01_P2.54mm_Vertical_SMD" H 8085 4265 50  0001 C CNN
 F 3 "~" H 8085 4265 50  0001 C CNN
 F 4 "-" H 8085 4265 50  0001 C CNN "LCSC#"
