File: Hardware/HunterCat-NFC/HunterCat-NFC.sch (KiCad schematic (older format))
At the start: 69 parts, among them J1 Battery, J2 Conn_01x06_Female, P1 USB_C_Plug_USB2.0, Q1 DMG3415U-7, SW1 RESET, SW2 GPIO, SW3 GPIO1, SW4 GPIO2, SW5 ON, U1 ATSAMD21E18A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

Commit message: update flash memmory
Parts:
- P1: symbol Connector:USB_C_Plug_USB2.0 -> HunterCat-NFC-rescue:USB_C_Plug_USB2.0-Connector
- U4: symbol Regulator_Linear:AP2112K-3.3 -> HunterCat-NFC-rescue:AP2112K-3.3-Regulator_Linear
Changed lines of the file:
@@
 $EndComp
 $Comp
-L Connector:USB_C_Plug_USB2.0 P1
+L HunterCat-NFC-rescue:USB_C_Plug_USB2.0-Connector P1
 U 1 1 5E5B360D
 P 4450 6595
@@
 	7850 470  7840 470
 $Comp
-L Regulator_Linear:AP2112K-3.3 U4
+L HunterCat-NFC-rescue:AP2112K-3.3-Regulator_Linear U4
 U 1 1 5E451F7B
 P 10405 4415
