File: Hardware/HunterCat-NFC/_autosave-HunterCat-NFC.kicad_sch (KiCad schematic)
At the start: 93 parts, among them J1 Battery, J2 Conn_01x06_Female, P1 USB_C_Plug_USB2.0, Q1 DMG3415U-7, SW1 RESET, SW2 GPIO, SW3 GPIO1, SW4 GPIO2, SW5 ON, U1 ATSAMD21E18A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

Commit message: Replace RP2040 pins labels
Parts:
- removed C1, C25: 0.1uF, Capacitor_SMD:C_0603_1608Metric_Pad1.05x0.95mm_HandSolder, symbol Device:C_Small
- removed C2: 1uF, Capacitor_SMD:C_0603_1608Metric_Pad1.05x0.95mm_HandSolder, symbol Device:C_Small
- removed R? (x2): 27, Resistor_SMD:R_0603_1608Metric, symbol Device:R_Small
- removed SW?: RESET, Button_Switch_SMD:SW_SPST_TL3342, symbol Switch:SW_Push
- removed U1: ATSAMD21E18A, Package_DFN_QFN:QFN-32-1EP_5x5mm_P0.5mm_EP3.6x3.6mm, symbol HunterCat-NFC-rescue:ATSAMD21E18A-Electronic_Cats
- removed U5: GD25Q16CEIGR, hunter-cat-nfc:PSON50P200X300X50-9N, symbol Memory_Flash:W25Q32JVSS
- added R22: 27, Resistor_SMD:R_0603_1608Metric, symbol Device:R_Small
- R21: value 10K -> 27; footprint Resistor_SMD:R_0603_1608Metric_Pad1.05x0.95mm_HandSolder -> Resistor_SMD:R_0603_1608Metric; LCSC# C15401 -> (none); manf# - -> (none); provedor LCSC -> (none)
- gave numbers to parts that had none: 21
Connections:
- net A0 is gone; now on net B_ADC: U1.38 (GPIO26_ADC0)
- net A1 is gone; now on net LED2: U1.39 (GPIO27_ADC1)
- net A2 is gone; now on net LED3: U1.40 (GPIO28_ADC2)
- net CIPO_0 is gone; now on net CLK: U1.27 (GPIO16)
- net COPI_1 is gone; now on net IRQ: U1.18 (GPIO15)
- net CS is gone; now on net RD+: R21.2
- net CS_1 is gone; now on net GPIO: U1.28 (GPIO17)
- net D13 is gone; now on net GPIO1: U1.32 (GPIO21)
- net D25 is gone; now on net LED1: U1.37 (GPIO25)
- net DIO0 is gone; now on net SCL: U1.7 (GPIO5)
- net DIO1 is gone; now on net SDA: U1.6 (GPIO4)
- net DIO5 is gone; now on net GPIO2: U1.34 (GPIO22)
- net SCK_1 is gone; now on net VEN: U1.17 (GPIO14)
- net +3V3: no longer R21.1
- net D+: now also R21.1
- net D-: now also R22.1
- net RD-: now also R22.2
- net SCL: no longer U1.5 (GPIO3)
- net SDA: no longer U1.4 (GPIO2)
- net A3: no longer names the net of U1.41 (GPIO29_ADC3)
- net COPI_0: no longer names the net of U1.30 (GPIO19)
- net D10: no longer names the net of U1.14 (GPIO11)
- net D11: no longer names the net of U1.15 (GPIO12)
- net D12: no longer names the net of U1.31 (GPIO20)
- net D24: no longer names the net of U1.36 (GPIO24)
- net D4: no longer names the net of U1.9 (GPIO7)
- net D5: no longer names the net of U1.11 (GPIO8)
- net D6: no longer names the net of U1.12 (GPIO9)
- net D9: no longer names the net of U1.13 (GPIO10)
- net DIO2: no longer names the net of U1.35 (GPIO23)
- net GPIO13: no longer names the net of U1.16 (GPIO13)
- net RF_RST: no longer names the net of U1.8 (GPIO6)
- net SCK_0: no longer names the net of U1.29 (GPIO18)
- no-connect marks 9 -> 19
Other:
- moved on the sheet: C10, C11, C12, C13, C14, C16, C18, C19, C20, C23, C24, C3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

Commit message: Assigned footprints
Parts:
- C1, C15: value 27pF -> (none); footprint Capacitor_SMD:C_0603_1608Metric -> (none)
- C10, C11: value 1nF/16V -> (none); footprint Capacitor_SMD:C_0603_1608Metric_Pad1.05x0.95mm_HandSolder -> (none)
- C12, C13: value 680pF -> (none); footprint Capacitor_SMD:C_0603_1608Metric_Pad1.05x0.95mm_HandSolder -> (none)
- C14, C18: value 100pF/50V -> (none); footprint Capacitor_SMD:C_0603_1608Metric_Pad1.05x0.95mm_HandSolder -> (none)
- C16, C23, C24: value 10uF -> (none); footprint Capacitor_SMD:C_0603_1608Metric_Pad1.05x0.95mm_HandSolder -> (none)
- C17, C21, C25, C26, C27, C28, C29, C30, C31, C32: value 0.1uF -> (none); footprint Capacitor_SMD:C_0603_1608Metric -> (none)
- C19, C20: value 120pF -> (none); footprint Capacitor_SMD:C_0603_1608Metric_Pad1.05x0.95mm_HandSolder -> (none)
- C2, C22: value 1uF -> (none); footprint Capacitor_SMD:C_0603_1608Metric -> (none)
- C3, C4: value 10pF -> (none); footprint Capacitor_SMD:C_0603_1608Metric_Pad1.05x0.95mm_HandSolder -> (none)
- C5, C6, C8: value 1uF -> (none); footprint Capacitor_SMD:C_0603_1608Metric_Pad1.05x0.95mm_HandSolder -> (none)
- C7, C9: value 100nF -> (none); footprint Capacitor_SMD:C_0603_1608Metric_Pad1.05x0.95mm_HandSolder -> (none)
- D1, D2, D3, D4: value LED -> (none); footprint LED_SMD:LED_0805_2012Metric_Pad1.15x1.40mm_HandSolder -> (none)
- D5: value MBR120 -> (none); footprint Diode_SMD:D_SOD-123F -> (none)
- F1: value 0.5A -> (none); footprint Fuse:Fuse_0603_1608Metric_Pad1.05x0.95mm_HandSolder -> (none)
- H1, H2, H3, H4: value MountingHole -> (none); footprint MountingHole:MountingHole_2.2mm_M2 -> (none)
- J1: value Battery -> (none); footprint Connector_PinSocket_2.54mm:PinSocket_2x01_P2.54mm_Vertical_SMD -> (none)
- J2: value Conn_01x06_Female -> (none); footprint Connector:Tag-Connect_TC2030-IDC-NL_2x03_P1.27mm_Vertical -> (none)
- L1, L2: value 160nH -> (none); footprint Inductor_SMD:L_0603_1608Metric_Pad1.05x0.95mm_HandSolder -> (none)
- L3: value L -> (none); footprint hunter-cat-nfc:NFC-antenna30.4x30.4mm -> (none)
- P1: value USB_C_Plug_USB2.0 -> (none); footprint Connectors:C393939 -> (none)
- Q1: value DMG3415U-7 -> (none); footprint Package_TO_SOT_SMD:SOT-23 -> (none)
- R1, R16, R2: value 10K -> (none); footprint Resistor_SMD:R_0603_1608Metric_Pad1.05x0.95mm_HandSolder -> (none)
- R10, R12, R17, R18, R4: value 1K -> (none); footprint Resistor_SMD:R_0603_1608Metric_Pad1.05x0.95mm_HandSolder -> (none)
- R11, R13: value 2k2 -> (none); footprint Resistor_SMD:R_0603_1608Metric_Pad1.05x0.95mm_HandSolder -> (none)
- R14, R15: value 3.24R -> (none); footprint Resistor_SMD:R_0603_1608Metric_Pad1.05x0.95mm_HandSolder -> (none)
- R19, R20, R3, R5, R6: value 100K -> (none); footprint Resistor_SMD:R_0603_1608Metric_Pad1.05x0.95mm_HandSolder -> (none)
- R21, R22: value 27 -> (none); footprint Resistor_SMD:R_0603_1608Metric -> (none)
- R23, R7: value 1K -> (none); footprint Resistor_SMD:R_0603_1608Metric -> (none)
- R24: value 10K -> (none); footprint Resistor_SMD:R_0603_1608Metric -> (none)
- R8, R9: value 5k1 -> (none); footprint Resistor_SMD:R_0603_1608Metric_Pad1.05x0.95mm_HandSolder -> (none)
- SW1: value RESET -> (none); footprint Button_Switch_SMD:SW_SPST_TL3342 -> (none)
- SW2: value GPIO -> (none); footprint Button_Switch_SMD:SW_SPST_TL3342 -> (none)
- SW3: value GPIO1 -> (none); footprint Button_Switch_SMD:SW_SPST_TL3342 -> (none)
- SW4: value GPIO2 -> (none); footprint Button_Switch_SMD:SW_SPST_TL3342 -> (none)
- SW5: value ON -> (none); footprint hunter-cat-nfc:Micro_interruptor_SPDT -> (none)
- SW6: value BOOT -> (none); footprint Button_Switch_SMD:SW_SPST_TL3342 -> (none)
- U1: value RP2040 -> (none); footprint badge_pwnCon:RP2040-QFN-56 -> (none)
- U2: value PN7150B0HN_C11002E-PN7150B0HN_C11002E -> (none); footprint Package_DFN_QFN:QFN-40-1EP_6x6mm_P0.5mm_EP4.6x4.6mm -> (none)
- U3: value MCP73831-3-OT -> (none); footprint Package_TO_SOT_SMD:SOT-23-5 -> (none)
- U4: value AP2112K-3.3 -> (none); footprint Package_TO_SOT_SMD:SOT-23-5 -> (none)
- U5: value W25Q16JV -> (none); footprint Package_SO:SOIC-8_5.275x5.275mm_P1.27mm -> (none)
- Y1: value 27.12Mhz -> (none); footprint Crystal:Crystal_SMD_2016-4Pin_2.0x1.6mm -> (none)
- Y2: value 12Mhz -> (none); footprint Crystal:Crystal_SMD_HC49-SD -> (none)
Other:
- moved on the sheet: C32, R24, U5
