File: Hardware/HunterCat-NFC/HunterCat-NFC.kicad_sch (KiCad schematic)
At the start: 69 parts, among them J1 Battery, J2 Conn_01x06_Female, P1 USB_C_Plug_USB2.0, Q1 DMG3415U-7, SW1 RESET, SW2 GPIO, SW3 GPIO1, SW4 GPIO2, SW5 ON, U1 ATSAMD21E18A, U2 PN7150B0HN_C11002E-PN7150B0HN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, U3 MCP73831-3-OT, U4 AP2112K-3.3, U5 GD25Q16CEIGR, Y1 27.12Mhz

Commit message: Replace RP2040 pins labels
Parts:
- removed C1, C25: 0.1uF, Capacitor_SMD:C_0603_1608Metric_Pad1.05x0.95mm_HandSolder, symbol Device:C_Small
- removed C2: 1uF, Capacitor_SMD:C_0603_1608Metric_Pad1.05x0.95mm_HandSolder, symbol Device:C_Small
- removed R21: 10K, Resistor_SMD:R_0603_1608Metric_Pad1.05x0.95mm_HandSolder, symbol Device:R_Small
- removed U1: ATSAMD21E18A, Package_DFN_QFN:QFN-32-1EP_5x5mm_P0.5mm_EP3.6x3.6mm, symbol HunterCat-NFC-rescue:ATSAMD21E18A-Electronic_Cats
- removed U5: GD25Q16CEIGR, hunter-cat-nfc:PSON50P200X300X50-9N, symbol Memory_Flash:W25Q32JVSS
- added C? (x10): 0.1uF, Capacitor_SMD:C_0603_1608Metric, symbol Device:C_Small
- added C? (x2): 1uF, Capacitor_SMD:C_0603_1608Metric, symbol Device:C_Small
- added C? (x2): 27pF, Capacitor_SMD:C_0603_1608Metric, symbol Device:C_Small
- added R? (x2): 1K, Resistor_SMD:R_0603_1608Metric, symbol Device:R_Small
- added R? (x2): 27, Resistor_SMD:R_0603_1608Metric, symbol Device:R_Small
- added R?: 10K, Resistor_SMD:R_0603_1608Metric, symbol Device:R_Small
- added SW?: BOOT, Button_Switch_SMD:SW_SPST_TL3342, symbol Switch:SW_Push
- added U?: W25Q16JV, Package_SO:SOIC-8_5.275x5.275mm_P1.27mm, symbol Memory_Flash:W25Q32JVZP
- added U?: RP2040, badge_pwnCon:RP2040-QFN-56, symbol PicoWAN-rescue:RP2040-MCU_RaspberryPi_and_Boards-PicoWAN-rescue-PicoWAN-rescue
- added Y?: 12Mhz, Crystal:Crystal_SMD_HC49-SD, symbol Device:Crystal_Small
Connections:
- net +3V3: now also C?.1, C?.1, C?.1, C?.1, C?.1, C?.1, C?.1, C?.1, C?.1, R?.1, U?.1 (IOVDD), U?.10 (IOVDD), U?.22 (IOVDD), U?.33 (IOVDD), U?.42 (IOVDD), U?.43 (ADC_AVDD), U?.44 (VREG_IN), U?.48 (USB_VDD), U?.49 (IOVDD), U?.8 (VCC)
- net B_ADC: now also U?.38 (GPIO26_ADC0)
- net CLK: now also U?.27 (GPIO16)
- net D+: now also R?.1
- net D-: now also R?.1
- net GND: now also C?.2, C?.2, C?.2, C?.2, C?.2, C?.2, C?.2, C?.2, C?.2, C?.2, C?.2, C?.2, C?.2, C?.2, SW?.1, U?.19 (TESTEN), U?.4 (GND), U?.57 (GND)
- net GPIO: now also U?.28 (GPIO17)
- net GPIO1: now also U?.32 (GPIO21)
- net GPIO2: now also U?.34 (GPIO22)
- net IRQ: now also U?.18 (GPIO15)
- net LED1: now also U?.37 (GPIO25)
- net LED2: now also U?.39 (GPIO27_ADC1)
- net LED3: now also U?.40 (GPIO28_ADC2)
- net RST: now also U?.26 (RUN)
- net SCL: now also U?.7 (GPIO5)
- net SDA: now also U?.6 (GPIO4)
- net SWCLK: now also U?.24 (SWCLK)
- net SWDIO: now also U?.25 (SWD)
- net VEN: now also U?.17 (GPIO14)
- new net: C?.1, U?.20 (XIN), Y?.1
- new net: C?.1, R?.1, Y?.2
- new net: R?.2, SW?.2
- new net: R?.2, U?.21 (XOUT)
- new net +1V2: C?.1, C?.1, C?.1, U?.23 (DVDD), U?.45 (VREG_VOUT), U?.50 (DVDD)
- new net QSPI_CS: R?.1, R?.2, U?.1 (~{CS}), U?.56 (QSPI_SS)
- new net QSPI_DATA0: U?.5 (DI(IO0)), U?.53 (QSPI_SD0)
- new net QSPI_DATA1: U?.2 (DO(IO1)), U?.55 (QSPI_SD1)
- new net QSPI_DATA2: U?.3 (IO2), U?.54 (QSPI_SD2)
- new net QSPI_DATA3: U?.51 (QSPI_SD3), U?.7 (IO3)
- new net QSPI_SCK: U?.52 (QSPI_SCLK), U?.6 (CLK)
- new net RD+: R?.2, U?.47 (USB_DP)
- new net RD-: R?.2, U?.46 (USB_DM)
- new net RX: U?.3 (GPIO1)
- new net TX: U?.2 (GPIO0)
- no-connect marks 8 -> 19
Other:
- note added: "FLASH"
- moved on the sheet: C10, C11, C12, C13, C14, C16, C18, C19, C20, C23, C24, C3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

Commit message: Assigned footprints
Parts:
- gave numbers to parts that had none: 23
Other:
- moved on the sheet: C32, R24, U5

Commit message: Replace RP2040 crystal footprint
Parts:
- removed R16: 10K, Resistor_SMD:R_0603_1608Metric_Pad1.05x0.95mm_HandSolder, symbol Device:R_Small
- C1, C15: value 27pF -> (none); footprint Capacitor_SMD:C_0603_1608Metric -> (none)
- C10, C11: value 1nF/16V -> (none); footprint Capacitor_SMD:C_0603_1608Metric_Pad1.05x0.95mm_HandSolder -> (none)
- C12, C13: value 680pF -> (none); footprint Capacitor_SMD:C_0603_1608Metric_Pad1.05x0.95mm_HandSolder -> (none)
- C14, C18: value 100pF/50V -> (none); footprint Capacitor_SMD:C_0603_1608Metric_Pad1.05x0.95mm_HandSolder -> (none)
- C16, C23, C24: value 10uF -> (none); footprint Capacitor_SMD:C_0603_1608Metric_Pad1.05x0.95mm_HandSolder -> (none)
- C17, C21, C25, C26, C27, C28, C29, C30, C31, C32: value 0.1uF -> (none); footprint Capacitor_SMD:C_0603_1608Metric -> (none)
- C19, C20: value 120pF -> (none); footprint Capacitor_SMD:C_0603_1608Metric_Pad1.05x0.95mm_HandSolder -> (none)
- C2, C22: value 1uF -> (none); footprint Capacitor_SMD:C_0603_1608Metric -> (none)
- C3, C4: value 10pF -> (none); footprint Capacitor_SMD:C_0603_1608Metric_Pad1.05x0.95mm_HandSolder -> (none)
- C5, C6, C8: value 1uF -> (none); footprint Capacitor_SMD:C_0603_1608Metric_Pad1.05x0.95mm_HandSolder -> (none)
- C7, C9: value 100nF -> (none); footprint Capacitor_SMD:C_0603_1608Metric_Pad1.05x0.95mm_HandSolder -> (none)
- D1, D2, D3, D4: value LED -> (none); footprint LED_SMD:LED_0805_2012Metric_Pad1.15x1.40mm_HandSolder -> (none)
- D5: value MBR120 -> (none); footprint Diode_SMD:D_SOD-123F -> (none)
- F1: value 0.5A -> (none); footprint Fuse:Fuse_0603_1608Metric_Pad1.05x0.95mm_HandSolder -> (none)
- H1, H2, H3, H4: value MountingHole -> (none); footprint MountingHole:MountingHole_2.2mm_M2 -> (none)
- J1: value Battery -> (none); footprint Connector_PinSocket_2.54mm:PinSocket_2x01_P2.54mm_Vertical_SMD -> (none)
- J2: value Conn_01x06_Female -> (none); footprint Connector:Tag-Connect_TC2030-IDC-NL_2x03_P1.27mm_Vertical -> (none)
- L1, L2: value 160nH -> (none); footprint Inductor_SMD:L_0603_1608Metric_Pad1.05x0.95mm_HandSolder -> (none)
- L3: value L -> (none); footprint hunter-cat-nfc:NFC-antenna30.4x30.4mm -> (none)
- P1: value USB_C_Plug_USB2.0 -> (none); footprint Connectors:C393939 -> (none)
- Q1: value DMG3415U-7 -> (none); footprint Package_TO_SOT_SMD:SOT-23 -> (none)
- R1, R2: value 10K -> (none); footprint Resistor_SMD:R_0603_1608Metric_Pad1.05x0.95mm_HandSolder -> (none)
- R10, R12, R17, R18, R4: value 1K -> (none); footprint Resistor_SMD:R_0603_1608Metric_Pad1.05x0.95mm_HandSolder -> (none)
- R11, R13: value 2k2 -> (none); footprint Resistor_SMD:R_0603_1608Metric_Pad1.05x0.95mm_HandSolder -> (none)
- R14, R15: value 3.24R -> (none); footprint Resistor_SMD:R_0603_1608Metric_Pad1.05x0.95mm_HandSolder -> (none)
- R19, R20, R3, R5, R6: value 100K -> (none); footprint Resistor_SMD:R_0603_1608Metric_Pad1.05x0.95mm_HandSolder -> (none)
- R21, R22: value 27 -> (none); footprint Resistor_SMD:R_0603_1608Metric -> (none)
- R23, R7: value 1K -> (none); footprint Resistor_SMD:R_0603_1608Metric -> (none)
- R24: value 10K -> (none); footprint Resistor_SMD:R_0603_1608Metric -> (none)
- R8, R9: value 5k1 -> (none); footprint Resistor_SMD:R_0603_1608Metric_Pad1.05x0.95mm_HandSolder -> (none)
- SW1: value RESET -> (none); footprint Button_Switch_SMD:SW_SPST_TL3342 -> (none)
- SW2: value GPIO -> (none); footprint Button_Switch_SMD:SW_SPST_TL3342 -> (none)
- SW3: value GPIO1 -> (none); footprint Button_Switch_SMD:SW_SPST_TL3342 -> (none)
- SW4: value GPIO2 -> (none); footprint Button_Switch_SMD:SW_SPST_TL3342 -> (none)
- SW5: value ON -> (none); footprint hunter-cat-nfc:Micro_interruptor_SPDT -> (none)
- SW6: value BOOT -> (none); footprint Button_Switch_SMD:SW_SPST_TL3342 -> (none)
- U1: value RP2040 -> (none); footprint badge_pwnCon:RP2040-QFN-56 -> (none)
- U2: value PN7150B0HN_C11002E-PN7150B0HN_C11002E -> (none); footprint Package_DFN_QFN:QFN-40-1EP_6x6mm_P0.5mm_EP4.6x4.6mm -> (none)
- U3: value MCP73831-3-OT -> (none); footprint Package_TO_SOT_SMD:SOT-23-5 -> (none)
- U4: value AP2112K-3.3 -> (none); footprint Package_TO_SOT_SMD:SOT-23-5 -> (none)
- U5: value W25Q16JV -> (none); footprint Package_SO:SOIC-8_5.275x5.275mm_P1.27mm -> (none)
- Y1: value 27.12Mhz -> (none); footprint Crystal:Crystal_SMD_2016-4Pin_2.0x1.6mm -> (none)
- Y2: value 12Mhz -> (none); footprint Crystal:Crystal_SMD_HC49-SD -> (none); manf# ABLS-12.000MHZ-B4-T -> ECS-120-18-30-JGN-TR; provedor (none) -> MOUSER
Connections:
- net at C23.1, SW5.2 (B), U4.1 (VIN): now also U4.3 (EN)

Commit message: change button for jumper force boot
Parts:
- removed R23: (no value), symbol Device:R_Small
- removed SW6: (no value), symbol Switch:SW_Push
- added JP?: BOOT, symbol Jumper:Jumper_2_Open
- C1, C15: value (none) -> 27pF; footprint (none) -> Capacitor_SMD:C_0603_1608Metric
- C10, C11: value (none) -> 1nF/16V; footprint (none) -> Capacitor_SMD:C_0603_1608Metric_Pad1.05x0.95mm_HandSolder
- C12, C13: value (none) -> 680pF; footprint (none) -> Capacitor_SMD:C_0603_1608Metric_Pad1.05x0.95mm_HandSolder
- C14, C18: value (none) -> 100pF/50V; footprint (none) -> Capacitor_SMD:C_0603_1608Metric_Pad1.05x0.95mm_HandSolder
- C16, C23, C24: value (none) -> 10uF; footprint (none) -> Capacitor_SMD:C_0603_1608Metric_Pad1.05x0.95mm_HandSolder
- C17, C21, C25, C26, C27, C28, C29, C30, C31, C32: value (none) -> 0.1uF; footprint (none) -> Capacitor_SMD:C_0603_1608Metric
- C19, C20: value (none) -> 120pF; footprint (none) -> Capacitor_SMD:C_0603_1608Metric_Pad1.05x0.95mm_HandSolder
- C2, C22: value (none) -> 1uF; footprint (none) -> Capacitor_SMD:C_0603_1608Metric
- C3, C4: value (none) -> 10pF; footprint (none) -> Capacitor_SMD:C_0603_1608Metric_Pad1.05x0.95mm_HandSolder
- C5, C6, C8: value (none) -> 1uF; footprint (none) -> Capacitor_SMD:C_0603_1608Metric_Pad1.05x0.95mm_HandSolder
- C7, C9: value (none) -> 100nF; footprint (none) -> Capacitor_SMD:C_0603_1608Metric_Pad1.05x0.95mm_HandSolder
- D1, D2, D3, D4: value (none) -> LED; footprint (none) -> LED_SMD:LED_0805_2012Metric_Pad1.15x1.40mm_HandSolder
- D5: value (none) -> MBR120; footprint (none) -> Diode_SMD:D_SOD-123F
- F1: value (none) -> 0.5A; footprint (none) -> Fuse:Fuse_0603_1608Metric_Pad1.05x0.95mm_HandSolder
- H1, H2, H3, H4: value (none) -> MountingHole; footprint (none) -> MountingHole:MountingHole_2.2mm_M2
- J1: value (none) -> Battery; footprint (none) -> Connector_PinSocket_2.54mm:PinSocket_2x01_P2.54mm_Vertical_SMD
- J2: value (none) -> Conn_01x06_Female; footprint (none) -> Connector:Tag-Connect_TC2030-IDC-NL_2x03_P1.27mm_Vertical
- L1, L2: value (none) -> 160nH; footprint (none) -> Inductor_SMD:L_0603_1608Metric_Pad1.05x0.95mm_HandSolder
- L3: value (none) -> L; footprint (none) -> hunter-cat-nfc:NFC-antenna30.4x30.4mm
- P1: value (none) -> USB_C_Plug_USB2.0; footprint (none) -> Connectors:C393939
- Q1: value (none) -> DMG3415U-7; footprint (none) -> Package_TO_SOT_SMD:SOT-23
- R1, R2: value (none) -> 10K; footprint (none) -> Resistor_SMD:R_0603_1608Metric_Pad1.05x0.95mm_HandSolder
- R10, R12: value (none) -> 1K; footprint (none) -> Resistor_SMD:R_0603_1608Metric_Pad1.05x0.95mm_HandSolder
- R11, R13: value (none) -> 2k2; footprint (none) -> Resistor_SMD:R_0603_1608Metric_Pad1.05x0.95mm_HandSolder
- R14, R15: value (none) -> 3.24R; footprint (none) -> Resistor_SMD:R_0603_1608Metric_Pad1.05x0.95mm_HandSolder
- R17, R18, R4: value (none) -> 330; footprint (none) -> Resistor_SMD:R_0603_1608Metric_Pad1.05x0.95mm_HandSolder
- R19, R20, R3, R5, R6: value (none) -> 100K; footprint (none) -> Resistor_SMD:R_0603_1608Metric_Pad1.05x0.95mm_HandSolder
- R21, R22: value (none) -> 27; footprint (none) -> Resistor_SMD:R_0603_1608Metric
- R24: value (none) -> 10K; footprint (none) -> Resistor_SMD:R_0603_1608Metric
- R7: value (none) -> 1K; footprint (none) -> Resistor_SMD:R_0603_1608Metric
- R8, R9: value (none) -> 5k1; footprint (none) -> Resistor_SMD:R_0603_1608Metric_Pad1.05x0.95mm_HandSolder
- SW1: value (none) -> RESET; footprint (none) -> Button_Switch_SMD:SW_SPST_TL3342
- SW2: value (none) -> GPIO; footprint (none) -> Button_Switch_SMD:SW_SPST_TL3342
- SW3: value (none) -> GPIO1; footprint (none) -> Button_Switch_SMD:SW_SPST_TL3342
- SW4: value (none) -> GPIO2; footprint (none) -> Button_Switch_SMD:SW_SPST_TL3342
- SW5: value (none) -> ON; footprint (none) -> hunter-cat-nfc:Micro_interruptor_SPDT
- U1: value (none) -> RP2040; footprint (none) -> RP2040:RP2040-QFN-56
- U2: value (none) -> PN7150B0HN_C11002E-PN7150B0HN_C11002E; footprint (none) -> Package_DFN_QFN:QFN-40-1EP_6x6mm_P0.5mm_EP4.6x4.6mm
- U3: value (none) -> MCP73831-3-OT; footprint (none) -> Package_TO_SOT_SMD:SOT-23-5
- U4: value (none) -> AP2112K-3.3; footprint (none) -> Package_TO_SOT_SMD:SOT-23-5
- U5: value (none) -> W25Q16JV; footprint (none) -> Package_SO:SOIC-8_5.275x5.275mm_P1.27mm
- Y1: value (none) -> 27.12Mhz; footprint (none) -> Crystal:Crystal_SMD_2016-4Pin_2.0x1.6mm
- Y2: value (none) -> 12Mhz; footprint (none) -> Crystal:Crystal_SMD_5032-2Pin_5.0x3.2mm
Connections:
- net GND: now also JP?.1 (A)
- net QSPI_CS: now also JP?.2 (B)

Commit message: update layout to 3.0v
Parts:
- removed J2: Conn_01x06_Female, Connector:Tag-Connect_TC2030-IDC-NL_2x03_P1.27mm_Vertical, symbol Connector:Conn_01x06_Female
- removed Y2: 12Mhz, Crystal:Crystal_SMD_5032-2Pin_5.0x3.2mm, symbol Device:Crystal_Small
- added Y2: 12Mhz, Crystal:Crystal_SMD_2520-4Pin_2.5x2.0mm, symbol Device:Crystal_GND2
- C10, C11, C12, C13, C14, C16, C18, C19, C20, C23, C24, C3, C4, C5, C6, C7, C8, C9: footprint Capacitor_SMD:C_0603_1608Metric_Pad1.05x0.95mm_HandSolder -> Capacitor_SMD:C_0603_1608Metric
- JP1: renamed from JP?; footprint (none) -> Jumper:SolderJumper-2_P1.3mm_Open_TrianglePad1.0x1.5mm
- R1, R10, R11, R12, R13, R14, R15, R17, R18, R19, R2, R20, R3, R4, R5, R6, R8, R9: footprint Resistor_SMD:R_0603_1608Metric_Pad1.05x0.95mm_HandSolder -> Resistor_SMD:R_0603_1608Metric
- U5: footprint Package_SO:SOIC-8_5.275x5.275mm_P1.27mm -> hunter-cat-nfc:W25Q16JVUUIQ; manf# W25Q16JVUXIQ -> W25Q16JVUUIQ
Connections:
- net GND: now also Y2.2
- net GPIO: now also U1.31 (GPIO20); no longer U1.28 (GPIO17)
- net GPIO2: now also U1.30 (GPIO19); no longer U1.34 (GPIO22)
- net IRQ: now also U1.29 (GPIO18); no longer U1.18 (GPIO15)
- net LED1: now also U1.11 (GPIO8); no longer U1.37 (GPIO25)
- net LED2: now also U1.12 (GPIO9); no longer U1.39 (GPIO27_ADC1)
- net LED3: now also U1.13 (GPIO10); no longer U1.40 (GPIO28_ADC2)
- net VEN: now also U1.28 (GPIO17); no longer U1.17 (GPIO14)
- net at C1.1, U1.20 (XIN): now also Y2.1
- net at C15.1, R7.1: now also Y2.3
- net CLK: no longer names the net of U2.40 (CLK_REQ)
- net CLK: no longer U1.27 (GPIO16)
- no-connect marks 19 -> 16
